File: kicad/Embedded_Project.kicad_pcb (KiCad board)
At the start: 2 copper layers, 66 parts, among them U10 GH39FKSW, U11 GH39FKSW, U12 GH39FKSW, U21 GH39FKSW, U22 GH39FKSW, U23 GH39FKSW, U24 GH39FKSW, U25 GH39FKSW, U26 GH39FKSW, U27 GH39FKSW, U37 GH39FKSW, U38 GH39FKSW, U39 GH39FKSW, U40 GH39FKSW, U50 GH39FKSW, U51 GH39FKSW, U52 GH39FKSW, U53 GH39FKSW, U54 GH39FKSW, U6 BlackPill_STLINK, U64 GH39FKSW, U66 GH39FKSW, U67 GH39FKSW, U68 GH39FKSW, U7 GH39FKSW, U8 GH39FKSW, U9 GH39FKSW

Commit message: upadate kicad pcb
Parts:
- removed AM0:1: LCtrl, voidswitch:VoidSwitch_1.25u_SMD
- removed AM0:10: 2, voidswitch:VoidSwitch_1u_SMD
- removed AM0:11: E, voidswitch:VoidSwitch_1u_SMD
- removed AM0:12: A, voidswitch:VoidSwitch_1u_SMD
- removed AM0:13: S, voidswitch:VoidSwitch_1u_SMD
- removed AM0:14: Z, voidswitch:VoidSwitch_1u_SMD
- removed AM0:15: LAlt, voidswitch:VoidSwitch_1.25u_SMD
- removed AM0:2: LShift, voidswitch:VoidSwitch_1u_SMD
- removed AM0:3: CAPS, voidswitch:VoidSwitch_1u_SMD
- removed AM0:4: Tab, voidswitch:VoidSwitch_1u_SMD
- removed AM0:5: ESC, voidswitch:VoidSwitch_1u_SMD
- removed AM0:6: Q, voidswitch:VoidSwitch_1u_SMD
- removed AM0:7: 1, voidswitch:VoidSwitch_1u_SMD
- removed AM0:8: W, voidswitch:VoidSwitch_1u_SMD
- removed AM0:9: 3, voidswitch:VoidSwitch_1u_SMD
- removed AM1:0: F, voidswitch:VoidSwitch_1u_SMD
- removed AM1:1: C, voidswitch:VoidSwitch_1u_SMD
- removed AM1:10: Y, voidswitch:VoidSwitch_1u_SMD
- removed AM1:14: LSpace, voidswitch:VoidSwitch_3u_SMD
- removed AM1:15: V, voidswitch:VoidSwitch_1u_SMD
- removed AM1:2: Fun, voidswitch:VoidSwitch_1.25u_SMD
- removed AM1:3: X, voidswitch:VoidSwitch_1u_SMD
- removed AM1:4: D, voidswitch:VoidSwitch_1u_SMD
- removed AM1:5: R, voidswitch:VoidSwitch_1u_SMD
- removed AM1:6: 4, voidswitch:VoidSwitch_1u_SMD
- removed AM1:8: T, voidswitch:VoidSwitch_1u_SMD
- removed H5, H6, H7, H8: MountingHole, MountingHole:MountingHole_3.2mm_M3_Pad
- removed REF**: 60pct, voidswitch:VoidSwitch_60_pct
- added Brd1: SSD1306, SSD1306:128x64OLED, F.Cu at (256.0, 86.8)
- added C1: 10u, Capacitor_SMD:C_0402_1005Metric, F.Cu at (330.2, 108.6)
- added C2: 10u, Capacitor_SMD:C_0402_1005Metric, F.Cu at (332.2, 108.6)
- added D1: B5819W, Diode_SMD:D_SOD-123, F.Cu at (336.4, 107.7)
- added F1: 500mA, Fuse:Fuse_0603_1608Metric, F.Cu at (331.2, 105.2)
- added FB1: 100 @ 100 MHz, Inductor_SMD:L_0805_2012Metric, F.Cu at (325.9, 107.5)
- added LDO1: AMS1117-3.3, Package_TO_SOT_SMD:SOT-223-3_TabPin2, F.Cu at (331.4, 115.5)
- U10, U11, U22, U23, U24, U25, U26, U27, U37, U38, U39, U40, U51, U52, U53, U54, U7, U8, U9: footprint Package_TO_SOT_SMD:SOT-23 -> PCM_marbastlib-xp-he:SW_MX_HE_0deg_1u
- U12: footprint Package_TO_SOT_SMD:SOT-23 -> PCM_marbastlib-xp-he:SW_MX_HE_0deg_1.75u
- U21: footprint Package_TO_SOT_SMD:SOT-23 -> PCM_marbastlib-xp-he:SW_MX_HE_0deg_1.5u
- U50: footprint Package_TO_SOT_SMD:SOT-23 -> PCM_marbastlib-xp-he:SW_MX_HE_0deg_2.25
- U6: value BlackPill_STLINK -> BlackPill
- U64, U66, U67: footprint Package_TO_SOT_SMD:SOT-23 -> PCM_marbastlib-xp-he:SW_MX_HE_0deg_1.25u
- U68: footprint Package_TO_SOT_SMD:SOT-23 -> PCM_marbastlib-xp-he:SW_MX_HE_0deg_3u
- moved H4 199.4 mm to (206.1, 206.9)
- moved H1 176.9 mm to (207.1, 80.1)
- moved R1 126.1 mm to (279.2, 75.3), turned to 90 degrees
- moved R2 125.7 mm to (279.2, 78.2), turned to -90 degrees
- moved U6 111.7 mm to (318.6, 88.7)
- moved U67 110.7 mm to (267.6, 196.2)
- moved AM1 108.3 mm to (323.9, 159.5)
- moved U38 92.7 mm to (270.0, 158.1)
- moved U26 92.7 mm to (322.4, 139.1)
- moved U50 92.7 mm to (229.5, 177.2)
- moved U11 92.6 mm to (293.8, 120.0)
- moved U8 92.6 mm to (236.7, 120.0)
- moved U10 92.6 mm to (274.8, 120.0)
- moved U12 92.6 mm to (224.8, 158.1)
- moved U21 92.6 mm to (222.4, 139.1)
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Connections:
- U6 pad 1: AM0:SELECT2 -> AM1
- U6 pad 10: AM0:SELECT3 -> unconnected-(U6-PA15-Pad10)
- U6 pad 16: AM0:SELECT1 -> AM0
- U6 pad 23: AM0:SELECT0 -> unconnected-(U6-PC14-Pad23)
- U6 pad 26: AM1:SELECT0 -> AM0:SELECT0
- U6 pad 27: AM1:SELECT1 -> AM0:SELECT1
- U6 pad 28: AM1:SELECT2 -> AM0:SELECT2
- U6 pad 29: AM1:SELECT3 -> AM0:SELECT3
- U6 pad 30: AM4 -> AM1:SELECT0
- U6 pad 31: PA5_SCK1 -> AM1:SELECT1
- U6 pad 32: PA6_MISO1 -> AM1:SELECT2
- U6 pad 33: PA7_MOSI1 -> AM1:SELECT3
Routing:
- net AM0:SELECT3: track 0.00 -> 200.7 mm, vias 0 -> 1
- net AM0:SELECT2: track 0.00 -> 195.6 mm, vias 0 -> 1
- net AM0:SELECT1: track 0.00 -> 175.1 mm, vias 0 -> 1
- net AM0:SELECT0: track 0.00 -> 173.0 mm, vias 0 -> 1
- net AM1:SELECT0: track 0.00 -> 129.6 mm, vias 0 -> 1
- net AM1:SELECT1: track 0.00 -> 128.4 mm, vias 0 -> 1
- net AM1:SELECT3: track 0.00 -> 114.1 mm, vias 0 -> 1
- net AM1:SELECT2: track 0.00 -> 113.8 mm, vias 0 -> 1
- net AM1: track 0.00 -> 109.3 mm
- net AM0: track 0.00 -> 107.2 mm
- net AM1:2: track 0.00 -> 70.3 mm
- net AM0:1: track 0.00 -> 63.4 mm
- net GND: track 0.00 -> 61.1 mm, vias 0 -> 9
- net AM1:14: track 0.00 -> 58.9 mm
- net +3V3: track 0.00 -> 57.2 mm, vias 0 -> 4
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- added copper zone on B.Cu, net (none)
- added copper zone on F.Cu, net (none)
- added copper zone on In2.Cu, net +3V3
- added copper zone on In1.Cu, net GND
Other:
- board outline added: 173.8 x 142.9 mm
- copper layers 2 -> 4
