File: kicad/Embedded_Project.kicad_sch (KiCad schematic)
At the start: 65 parts, among them U10 GH39FKSW, U11 GH39FKSW, U12 GH39FKSW, U21 GH39FKSW, U22 GH39FKSW, U23 GH39FKSW, U24 GH39FKSW, U25 GH39FKSW, U26 GH39FKSW, U27 GH39FKSW, U37 GH39FKSW, U38 GH39FKSW, U39 GH39FKSW, U40 GH39FKSW, U50 GH39FKSW, U51 GH39FKSW, U52 GH39FKSW, U53 GH39FKSW, U54 GH39FKSW, U6 BlackPill_STLINK, U64 GH39FKSW, U66 GH39FKSW, U67 GH39FKSW, U68 GH39FKSW, U7 GH39FKSW, U8 GH39FKSW, U9 GH39FKSW

Commit message: upadate kicad pcb
Parts:
- added Brd1: SSD1306, SSD1306:128x64OLED, symbol SSD1306-128x64_OLED:SSD1306
- added C1, C2: 10u, Capacitor_SMD:C_0402_1005Metric, symbol Device:C_Small
- added D1: B5819W, Diode_SMD:D_SOD-123, symbol Device:D_Schottky_Small
- added F1: 500mA, Fuse:Fuse_0603_1608Metric, symbol Device:Fuse_Small
- added FB1: 100 @ 100 MHz, Inductor_SMD:L_0805_2012Metric, symbol Device:Ferrite_Bead_Small
- added LDO1: AMS1117-3.3, Package_TO_SOT_SMD:SOT-223-3_TabPin2, symbol Regulator_Linear:AMS1117-3.3
- H1, H2, H3, H4, H5, H6, H7, H8: now left out of the parts list
- U10, U11, U22, U23, U24, U25, U26, U27, U37, U38, U39, U40, U51, U52, U53, U54, U7, U8, U9: footprint Package_TO_SOT_SMD:SOT-23 -> PCM_marbastlib-xp-he:SW_MX_HE_0deg_1u
- U12: footprint Package_TO_SOT_SMD:SOT-23 -> PCM_marbastlib-xp-he:SW_MX_HE_0deg_1.75u
- U21: footprint Package_TO_SOT_SMD:SOT-23 -> PCM_marbastlib-xp-he:SW_MX_HE_0deg_1.5u
- U50: footprint Package_TO_SOT_SMD:SOT-23 -> PCM_marbastlib-xp-he:SW_MX_HE_0deg_2.25
- U64, U66, U67: footprint Package_TO_SOT_SMD:SOT-23 -> PCM_marbastlib-xp-he:SW_MX_HE_0deg_1.25u
- U68: footprint Package_TO_SOT_SMD:SOT-23 -> PCM_marbastlib-xp-he:SW_MX_HE_0deg_3u
Connections:
- net AM4 is gone; now on net AM1:SELECT0: U6.30 (PA4)
- net PA5_SCK1 is gone; now on net AM1:SELECT1: U6.31 (PA5)
- net PA6_MISO1 is gone; now on net AM1:SELECT2: U6.32 (PA6)
- net PA7_MOSI1 is gone; now on net AM1:SELECT3: U6.33 (PA7)
- net +3.3V_QWIIC: now also Brd1.2 (VCC)
- net +3V3: now also C2.1, LDO1.2 (VO)
- net +5V: now also D1.2 (A)
- net AM0: now also U6.16 (PB8)
- net AM0:SELECT0: now also U6.26 (PA0); no longer U6.23 (PC14)
- net AM0:SELECT1: now also U6.27 (PA1); no longer U6.16 (PB8)
- net AM0:SELECT2: now also U6.28 (PA2); no longer U6.1 (PB12)
- net AM0:SELECT3: now also U6.29 (PA3); no longer U6.10 (PA15)
- net AM1: now also U6.1 (PB12)
- net AM1:SELECT0: no longer U6.26 (PA0)
- net AM1:SELECT1: no longer U6.27 (PA1)
- net AM1:SELECT2: no longer U6.28 (PA2)
- net AM1:SELECT3: no longer U6.29 (PA3)
- net GND: now also Brd1.1 (GND), C1.2, C2.2, LDO1.1 (GND)
- net PB6_SCL1: now also Brd1.3 (SCL)
- net PB7_SDA1: now also Brd1.4 (SDA)
- new net: C1.1, FB1.1, LDO1.3 (VI)
- new net: F1.2, FB1.2
- new net: D1.1 (K), F1.1
Other:
- note added: "Capslock"
- note added: "Sensor 3.3V LDO"
- note added: "Tabs"
- note removed: "Tab"
