File: kicad/keypad.kicad_sch (KiCad schematic)
At the start: 80 parts, among them U6 BlackPill_STLINK

Commit message: updated minor errors
Connections:
- net FLASH_CS: no longer names the net of U6.17 (PB9)
- net PWR_SENSE: no longer names the net of U6.37 (PB10)
Other:
- note removed: "Power Attachment Detection"
Changed lines of the file:
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@@
 		)
 	)
-	(text "Power Attachment\nDetection"
-		(exclude_from_sim no)
-		(at 101.346 159.512 0)
-		(effects
-			(font
-				(size 1.27 1.27)
-			)
-			(justify right bottom)
-		)
-	)
 	(text "MUX"
 		(exclude_from_sim no)
@@
 	)
 	(junction
-		(at 290.83 99.06)
-		(diameter 0)
-		(color 0 0 0 0)
-	)
-	(junction
 		(at 203.2 190.5)
 		(diameter 0)
@@
 	(wire
 		(pts
-			(xy 288.29 99.06) (xy 290.83 99.06)
+			(xy 288.29 99.06) (xy 293.37 99.06)
 		)
 		(stroke
@@
 	(wire
 		(pts
-			(xy 290.83 99.06) (xy 293.37 99.06)
-		)
-		(stroke
-			(width 0)
-			(type default)
-		)
-	)
-	(wire
-		(pts
 			(xy 120.65 222.25) (xy 127 222.25)
 		)
@@
 	(wire
 		(pts
-			(xy 290.83 92.71) (xy 290.83 99.06)
-		)
-		(stroke
-			(width 0)
-			(type default)
-		)
-	)
-	(wire
-		(pts
 			(xy 226.06 200.66) (xy 240.03 200.66)
 		)
@@
 		)
 	)
-	(global_label "FLASH_CS"
-		(shape input)
-		(at 69.85 153.67 0)
-		(fields_autoplaced yes)
-		(effects
-			(font
-				(size 1.27 1.27)
-			)
-			(justify left)
-		)
-		(property "Intersheetrefs" "${INTERSHEET_REFS}"
-			(at -3.81 -5.08 0)
-			(effects
-				(font
-					(size 1.27 1.27)
-				)
-				(hide yes)
-			)
-		)
-	)
 	(global_label "AM0:5"
 		(shape input)
@@
 		)
 	)
-	(global_label "PWR_SENSE"
-		(shape input)
-		(at 69.85 156.21 0)
-		(fields_autoplaced yes)
-		(effects
-			(font
-				(size 1.27 1.27)
-			)
-			(justify left)
-		)
-		(property "Intersheetrefs" "${INTERSHEET_REFS}"
-			(at -16.51 -5.08 0)
-			(effects
-				(font
-					(size 1.27 1.27)
-				)
-				(hide yes)
-			)
-		)
-	)
 	(global_label "OLED_SDA"
 		(shape input)
@@
 					(unit 1)
 				)
-			)
-		)
-	)
-	(symbol
-		(lib_id "power:PWR_FLAG")
-		(at 290.83 92.71 0)
-		(unit 1)
-		(exclude_from_sim no)
-		(in_bom yes)
-		(on_board yes)
-		(dnp no)
-		(property "Reference" "#FLG01"
-			(at 290.83 90.805 0)
-			(effects
-				(font
-					(size 1.27 1.27)
-				)
-				(hide yes)
-			)
-		)
-		(property "Value" "PWR_FLAG"
-			(at 290.83 88.3158 0)
-			(effects
-				(font
-					(size 1.27 1.27)
-				)
-			)
-		)
-		(property "Footprint" ""
-			(at 290.83 92.71 0)
-			(effects
-				(font
-					(size 1.27 1.27)
-				)
-				(hide yes)
-			)
-		)
-		(property "Datasheet" "~"
-			(at 290.83 92.71 0)
-			(effects
-				(font
-					(size 1.27 1.27)
-				)
-				(hide yes)
-			)
-		)
-		(property "Description" ""
-			(at 290.83 92.71 0)
-			(effects
-				(font
-					(size 1.27 1.27)
-				)
-			)
-		)
-		(pin "1"
-		)
-		(instances
-			(project "keypad"
-				(path "/3cbe17a3-a42e-41fd-afb0-bb7258c20710"
-					(reference "#FLG01")
-					(unit 1)
-				)
